File: OpenPauw.kicad_pcb (KiCad board)
At the start: 2 copper layers, 18 parts, among them J1 Conn_01x01, J2 Conn_01x01, J3 Conn_01x01, J4 Conn_01x01, J5 Conn_01x04, U1 MAX328EPE+, U2 MAX328EPE+, U3 MAX328EPE+, U4 MAX328EPE+, U5 Adafruit-Feather-RP2040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

Commit message: New layout
Parts:
- added  : LOGO, LOGO, F.Cu at (118.7, 103.2)
- added  : LOGO, LOGO, F.Cu at (118.5, 38.3)
- moved C3 149.0 mm to (206.7, 51.1), turned to -90 degrees
- moved C2 128.7 mm to (192.3, 55.0), turned to -90 degrees
- moved D1 120.9 mm to (193.7, 43.7), turned to 180 degrees
- moved L1 116.0 mm to (179.4, 43.9)
- moved U6 110.5 mm to (169.8, 48.5), turned to 180 degrees
- moved R2 103.3 mm to (181.8, 59.5), turned to 90 degrees
- moved C1 98.1 mm to (159.4, 49.1), turned to -90 degrees
- moved R1 97.1 mm to (174.9, 55.9), turned to 180 degrees
- moved J5 56.4 mm to (134.4, 39.7), turned to 180 degrees
- moved U5 54.0 mm to (188.1, 78.6), turned to 180 degrees
- moved U1 38.6 mm to (145.9, 47.7), turned to -90 degrees
- moved U2 21.9 mm to (146.0, 60.9), turned to -90 degrees
- moved U4 18.2 mm to (145.8, 87.6), turned to -90 degrees
- moved U3 9.51 mm to (146.0, 74.3), turned to -90 degrees
Routing:
- net +15V: track 0.00 -> 187.2 mm, vias 0 -> 1
- net +5V: track 0.00 -> 108.9 mm
- net A2: track 0.00 -> 96.5 mm
- net A1: track 0.00 -> 96.4 mm
- net EN_U1: track 0.00 -> 96.3 mm
- net EN_U2: track 0.00 -> 96.1 mm
- net EN_U4: track 0.00 -> 95.8 mm
- net EN_U3: track 0.00 -> 95.8 mm
- net A0: track 0.00 -> 95.6 mm, vias 0 -> 2
- net PAD_D: track 0.00 -> 58.3 mm
- net PAD_A: track 0.00 -> 58.3 mm
- net PAD_C: track 0.00 -> 58.3 mm
- net PAD_B: track 0.00 -> 58.3 mm
- net Net-(U6-FB): track 0.00 -> 41.2 mm
- net Net-(D1-A): track 0.00 -> 33.9 mm, vias 0 -> 1
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- added copper zone on B.Cu, net GND
- added copper zone on F.Cu, net GND
Other:
- board outline added: 126.7 x 80.3 mm

Commit message: Fixed all DRC errors
Routing:
- net GND: track 0.00 -> 15.1 mm, vias 0 -> 5
- net A0: track 95.6 -> 93.4 mm
- net +15V: track 187.2 -> 185.2 mm, vias 1 -> 2
- net +5V: track 108.9 -> 110.8 mm

Commit message: New JST
Parts:
- J5: footprint Connector_JST:JST_GH_BM04B-GHS-TBT_1x04-1MP_P1.25mm_Vertical -> Connector_JST:JST_PH_B4B-PH-SM4-TB_1x04-1MP_P2.00mm_Vertical
- moved J5 3.05 mm to (134.2, 36.6)
Routing:
- net GND: track 15.1 -> 0.00 mm, vias 5 -> 0
- net PAD_B: track 58.3 -> 61.8 mm
- net PAD_C: track 58.3 -> 61.6 mm
- net PAD_D: track 58.3 -> 60.8 mm
- net PAD_A: track 58.3 -> 60.8 mm
